File: proyecto2.kicad_pcb (KiCad board)
At the start: 2 copper layers, 38 parts, among them Q1 2N2219, SW1 SW_SPDT, SW10 SW_Push, SW11 SW_Push, SW12 SW_Push, SW13 SW_Push, SW14 SW_Push, SW2 SW_Push, SW3 SW_Push, SW4 SW_Push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

Commit message: Add files via upload
Parts:
- removed U1: NE555D, Package_SO:SOIC-8_3.9x4.9mm_P1.27mm
- added U2: NE555P, Package_DIP:DIP-8_W7.62mm, F.Cu at (209.0, 120.5)
- moved Q1 36.4 mm to (254.9, 117.0)
- moved BZ1 36.3 mm to (246.8, 133.5)
- moved Agudo1 18.9 mm to (182.0, 124.6)
- moved Grave1 18.9 mm to (182.0, 115.6)
- moved R1 18.7 mm to (222.8, 120.5)
- moved SW1 17.1 mm to (193.5, 122.5)
- moved FAB1 15.0 mm to (120.6, 90.5)
- moved RE1 15.0 mm to (60.4, 90.5)
- moved REB1 15.0 mm to (45.7, 90.5)
- moved SW2 15.0 mm to (31.5, 95.8)
- moved SW4 15.0 mm to (61.0, 95.8)
- moved Do1 15.0 mm to (31.3, 91.0)
- moved DOMAJ1 15.0 mm to (214.5, 91.5)
- moved FA1 15.0 mm to (105.8, 90.3)
- moved LA1 15.0 mm to (168.2, 91.0)
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Routing:
- net Earth: track 0.00 -> 514.6 mm
- net Net-(U2-OUT): track 0.00 -> 502.7 mm
- net Net-(SW10-Pad2): track 0.00 -> 190.0 mm
- net Net-(BT1-+): track 0.00 -> 113.3 mm
- net Net-(BZ1--): track 0.00 -> 58.3 mm
- net Net-(Q1-B): track 0.00 -> 37.0 mm
- net Net-(SW1-A): track 1.89 -> 35.2 mm
- net Net-(SW1-B): track 0.00 -> 23.6 mm
- net Net-(U2-CONT): track 0.00 -> 19.4 mm
- net Net-(MI1-Pad1): track 0.00 -> 12.3 mm
- net Net-(MIB1-Pad1): track 0.00 -> 12.3 mm
- net Net-(FA1-Pad1): track 0.00 -> 12.3 mm
- net Net-(FAB1-Pad1): track 0.00 -> 12.3 mm
- net Net-(RE1-Pad1): track 0.00 -> 12.0 mm
- net Net-(SIB1-Pad1): track 0.00 -> 12.0 mm
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- added copper zone on F.Cu, net Earth
Other:
- board text added: "Electrica I | BN"
- board text added: "Veronica Fabiola Canas Flores"
- board text added: "Wagner Norwell Perez Castaneda | 25000167"
- board text added: "| 25001710"

Commit message: Add files via upload
Other:
- board outline added: 242.6 x 78.7 mm
