File: proyecto2.kicad_sch (KiCad schematic)
At the start: 38 parts, among them Q1 2N2219, SW1 SW_SPDT, SW10 SW_Push, SW11 SW_Push, SW12 SW_Push, SW13 SW_Push, SW14 SW_Push, SW2 SW_Push, SW3 SW_Push, SW4 SW_Push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

Commit message: Add files via upload
Parts:
- removed U1: NE555D, Package_SO:SOIC-8_3.9x4.9mm_P1.27mm, symbol Timer:NE555D
- added U2: NE555P, Package_DIP:DIP-8_W7.62mm, symbol Timer:NE555P
Connections:
- net Earth: now also U2.1 (GND)
- net at BT1.1 (+), BZ1.1 (+), C1.2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: now also U2.4 (~{RST}), U2.8 (VCC)
- net at C2.2: now also U2.5 (CONT)
- net at SW1.1 (A): now also U2.2 (TRIG), U2.6 (THRES), U2.7 (DISCH)
- net at R2.1: now also U2.3 (OUT)
Changed lines of the file:
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@@
 	)
 	(junction
-		(at 125.73 73.66)
-		(diameter 0)
-		(color 0 0 0 0)
-	)
-	(junction
 		(at 182.88 114.3)
 		(diameter 0)
@@
 	)
 	(junction
+		(at 125.73 73.66)
+		(diameter 0)
+		(color 0 0 0 0)
+	)
+	(junction
 		(at 104.14 133.35)
 		(diameter 0)
@@
 	)
 	(junction
+		(at 113.03 97.79)
+		(diameter 0)
+		(color 0 0 0 0)
+	)
+	(junction
 		(at 78.74 133.35)
 		(diameter 0)
@@
 	)
 	(junction
-		(at 113.03 97.79)
-		(diameter 0)
-		(color 0 0 0 0)
-	)
-	(junction
 		(at 161.29 114.3)
 		(diameter 0)
@@
 	(wire
 		(pts
-			(xy 113.03 97.79) (xy 113.03 100.33)
+			(xy 113.03 92.71) (xy 113.03 97.79)
 		)
 		(stroke
@@
 	(wire
 		(pts
-			(xy 213.36 133.35) (xy 223.52 133.35)
+			(xy 113.03 97.79) (xy 113.03 100.33)
 		)
 		(stroke
@@
 	(wire
 		(pts
-			(xy 149.86 114.3) (xy 161.29 114.3)
+			(xy 213.36 133.35) (xy 223.52 133.35)
 		)
 		(stroke
@@
 	(wire
 		(pts
-			(xy 127 124.46) (xy 127 125.73)
+			(xy 149.86 114.3) (xy 161.29 114.3)
 		)
 		(stroke
@@
 	(wire
 		(pts
-			(xy 133.35 95.25) (xy 135.89 95.25)
+			(xy 127 124.46) (xy 127 125.73)
 		)
 		(stroke
@@
 	(wire
 		(pts
-			(xy 167.64 78.74) (xy 167.64 90.17)
+			(xy 133.35 95.25) (xy 135.89 95.25)
 		)
 		(stroke
@@
 	(wire
 		(pts
-			(xy 113.03 92.71) (xy 113.03 97.79)
+			(xy 167.64 78.74) (xy 167.64 90.17)
 		)
 		(stroke
@@
 	)
 	(symbol
+		(lib_id "Timer:NE555P")
+		(at 123.19 95.25 0)
+		(unit 1)
+		(body_style 1)
+		(exclude_from_sim no)
+		(in_bom yes)
+		(on_board yes)
+		(in_pos_files yes)
+		(dnp no)
+		(fields_autoplaced yes)
+		(property "Reference" "U2"
+			(at 135.89 88.8298 0)
+			(show_name no)
+			(do_not_autoplace no)
+			(effects
+				(font
+					(size 1.27 1.27)
+				)
+			)
+		)
+		(property "Value" "NE555P"
+			(at 135.89 91.3698 0)
+			(show_name no)
+			(do_not_autoplace no)
+			(effects
+				(font
+					(size 1.27 1.27)
+				)
+			)
+		)
+		(property "Footprint" "Package_DIP:DIP-8_W7.62mm"
+			(at 123.19 119.38 0)
+			(hide yes)
+			(show_name no)
+			(do_not_autoplace no)
+			(effects
+				(font
+					(size 1.27 1.27)
+				)
+			)
+		)
+		(property "Datasheet" "http://www.ti.com/lit/ds/symlink/ne555.pdf"
+			(at 123.19 121.92 0)
+			(hide yes)
+			(show_name no)
+			(do_not_autoplace no)
+			(effects
+				(font
+					(size 1.27 1.27)
+				)
+			)
+		)
+		(property "Description" "Precision Timers, 555 compatible, PDIP-8"
+			(at 123.19 116.84 0)
+			(hide yes)
+			(show_name no)
+			(do_not_autoplace no)
+			(effects
+				(font
+					(size 1.27 1.27)
+				)
+			)
+		)
+		(pin "4"
+		)
+		(pin "1"
+		)
+		(pin "3"
+		)
+		(pin "8"
+		)
+		(pin "5"
+		)
+		(pin "2"
+		)
+		(pin "6"
+		)
+		(pin "7"
+		)
+		(instances
+			(project "proyecto2"
+				(path "/2acde91a-b0f1-4d66-bbdb-3257e67dbab9"
+					(reference "U2")
+					(unit 1)
+				)
+			)
+		)
+	)
+	(symbol
 		(lib_id "Transistor_BJT:2N2219")
 		(at 165.1 95.25 0)
@@
 					(unit 1)
 				)
-			)
-		)
-	)
-	(symbol
-		(lib_id "Timer:NE555D")
-		(at 123.19 95.25 0)
-		(unit 1)
-		(body_style 1)
-		(exclude_from_sim no)
-		(in_bom yes)
-		(on_board yes)
-		(in_pos_files yes)
-		(dnp no)
-		(property "Reference" "U1"
-			(at 124.206 95.504 0)
-			(show_name no)
-			(do_not_autoplace no)
-			(effects
-				(font
-					(size 1.27 1.27)
-				)
-				(justify right)
-			)
-		)
-		(property "Value" "NE555D"
-			(at 120.0719 105.41 0)
-			(show_name no)
-			(do_not_autoplace no)
-			(effects
-				(font
-					(size 1.27 1.27)
-				)
-				(justify right)
-			)
-		)
-		(property "Footprint" "Package_SO:SOIC-8_3.9x4.9mm_P1.27mm"
-			(at 123.19 119.38 0)
-			(hide yes)
-			(show_name no)
-			(do_not_autoplace no)
-			(effects
-				(font
-					(size 1.27 1.27)
-				)
-			)
-		)
-		(property "Datasheet" "http://www.ti.com/lit/ds/symlink/ne555.pdf"
-			(at 123.19 121.92 0)
-			(hide yes)
-			(show_name no)
-			(do_not_autoplace no)
-			(effects
-				(font
-					(size 1.27 1.27)
-				)
-			)
-		)
-		(property "Description" "Precision Timers, 555 compatible, SOIC-8"
-			(at 123.19 116.84 0)
-			(hide yes)
-			(show_name no)
-			(do_not_autoplace no)
-			(effects
-				(font
-					(size 1.27 1.27)
-				)
-			)
-		)
-		(pin "5"
-		)
-		(pin "8"
-		)
-		(pin "2"
-		)
-		(pin "3"
-		)
-		(pin "7"
-		)
-		(pin "6"
-		)
-		(pin "1"
-		)
-		(pin "4"
-		)
-		(instances
-			(project "proyecto2"
-				(path "/2acde91a-b0f1-4d66-bbdb-3257e67dbab9"
-					(reference "U1")
-					(unit 1)
-				)

Commit message: Add files via upload
Changed lines of the file:
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@@
-	)
-	(junction
-		(at 99.06 88.9)
-		(diameter 0)
-		(color 0 0 0 0)
 	)
 	(junction
@@
 	(wire
 		(pts
+			(xy 99.06 77.47) (xy 99.06 88.9)
+		)
+		(stroke
+			(width 0)
+			(type default)
+		)
+	)
+	(wire
+		(pts
 			(xy 182.88 133.35) (xy 193.04 133.35)
 		)
@@
 	(wire
 		(pts
-			(xy 99.06 77.47) (xy 99.06 88.9)
-		)
-		(stroke
-			(width 0)
-			(type default)
-		)
-	)
-	(wire
-		(pts
 			(xy 144.78 80.01) (xy 144.78 73.66)
 		)
@@
 		)
 		(stroke
-			(width 0)
-			(type default)
-		)
-	)
-	(wire
-		(pts
-			(xy 99.06 88.9) (xy 99.06 90.17)
-		)
-		(stroke
